File: unonano.brd (EAGLE design)
At the start: 71.1 x 90 mm, 25 parts, among them J13 AVR_SPI_PROG_3X2NS, U1 ATTINY85-20P

Commit message: lookin good
Parts:
- removed SJ1, SJ2, SJ3: (no value), jumper:SJ
- added ARDUINO_ISP, ICP_FOR_BIG, ICP_FOR_SMALL: (no value), jumper:SJ
- moved J12 125.7 mm to (66.8, 64.5), turned to 90 degrees
- moved J19 124.8 mm to (60.5, 26.7), turned to 90 degrees
- moved J18 124.1 mm to (65.5, 26.7), turned to 90 degrees
- moved J11 124.0 mm to (69.3, 64.5), turned to 90 degrees
- moved J17 119.6 mm to (63.0, 26.7), turned to 90 degrees
- moved J10 116.6 mm to (69.3, 59.3), turned to 270 degrees
- moved J16 116.0 mm to (47.2, 34.3), turned to 270 degrees
- moved J9 112.3 mm to (66.8, 59.4), turned to 270 degrees
- moved J15 111.6 mm to (44.7, 34.3), turned to 270 degrees
- moved J14 107.2 mm to (42.2, 34.3), turned to 270 degrees
- moved J13 106.0 mm to (71.9, 33.5), turned to 270 degrees
- moved J6 102.2 mm to (30.2, 77.2), turned to 270 degrees
- moved U1 100.4 mm to (53.8, 30.5), turned to 270 degrees
- moved J5 99.5 mm to (32.8, 77.2), turned to 270 degrees
- moved J2 89.5 mm to (39.4, 74.9), turned to 270 degrees
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Connections:
- removed net PWM_R: U$1.D10
- removed net TNY03: U1.2
- removed net TNY04: U1.3
- removed net TNYRST: U1.1
- net AVRRST: now also ICP_FOR_BIG.2, ICP_FOR_SMALL.2; no longer SJ1.2, SJ2.2
- net BIGRST: now also ICP_FOR_BIG.1; no longer SJ1.1
- net D10: now also ARDUINO_ISP.1, U$1.D10; no longer SJ3.1
- net TINY03: now also U1.2
- net TINY04: now also U1.3
- net TINYRST: now also ARDUINO_ISP.2, ICP_FOR_SMALL.1, U1.1; no longer SJ2.1, SJ3.2
Routing:
- net D13: track 0.00 -> 19.7 mm
- net D12: track 0.00 -> 19.7 mm
- net D11: track 0.00 -> 19.7 mm
- net BIGRST: track 0.00 -> 15.5 mm
- net VIN: track 0.00 -> 13.0 mm
- net +3.3V: track 0.00 -> 13.0 mm
- net A4: track 0.00 -> 12.9 mm
- net A2: track 0.00 -> 12.9 mm
- net A0: track 0.00 -> 12.9 mm
- net A5: track 0.00 -> 12.9 mm
- net A3: track 0.00 -> 12.9 mm
- net TX: track 0.00 -> 11.8 mm
- net D5: track 0.00 -> 11.8 mm
- net D4: track 0.00 -> 11.8 mm
- net D3: track 0.00 -> 11.8 mm
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- removed copper zone on layer 1, net +5V
- removed copper zone on layer 16, net GND
Other:
- board size 71.1 x 90 mm -> 100 x 100 mm
- board text removed: "+3.3V"
- board text removed: "+5V"
- board text removed: "+5v"
- board text removed: "??"
- board text removed: "???"
- board text removed: "A0"
- board text removed: "A1"
- board text removed: "A2"
- board text removed: "A3"
- board text removed: "A4"
- board text removed: "A5"
- board text removed: "A6"
- board text removed: "A7"
- board text removed: "AREF"
- board text removed: "BACK"
- board text removed: "D10"
- board text removed: "D11"
- board text removed: "D12"
- board text removed: "D13"
- board text removed: "D2"
- board text removed: "D3"
- board text removed: "D4"
- board text removed: "D5"
- board text removed: "D6"
- board text removed: "D7"
- board text removed: "D8"
- board text removed: "D9"
- board text removed: "Derick Louie"
- board text removed: "EB"
- board text removed: "EF"
- board text removed: "EL"
- board text removed: "ER"
- board text removed: "FRONT"
- board text removed: "GND"
- board text removed: "Input / Triplet Sheild"
- board text removed: "Kevin Kellar"
- board text removed: "LEFT"
- board text removed: "PWM_L"
- board text removed: "PWM_R"
- board text removed: "RIGHT"
- board text removed: "RST"
- board text removed: "RX"
- board text removed: "SBL"
- board text removed: "SBR"
- board text removed: "SFL"
- board text removed: "SFR"
- board text removed: "SLB"
- board text removed: "SLF"
- board text removed: "SRB"
- board text removed: "SRF"
- board text removed: "TRIG"
- board text removed: "TX"
- board text removed: "VIN"
