File: multishift.brd (EAGLE design)
At the start: 100 x 100 mm, 184 parts, among them J13 AVR_SPI_PROG_3X2NS, U1 ATTINY85-20P

Commit message: multishift so so close
Parts:
- removed MOSFET-15: (no value), SparkFun-Connectors:1X03
- removed OUT_10_PULLDOWN_RES, OUT_10_PULLUP_RES, OUT_11_PULLDOWN_RES, OUT_11_PULLUP_RES, OUT_12_PULLDOWN_RES, OUT_12_PULLUP_RES, OUT_13_PULLDOWN_RES, OUT_13_PULLUP_RES, OUT_14_PULLDOWN_RES, OUT_14_PULLUP_RES, OUT_15_PULLDOWN_RES, OUT_15_PULLUP_RES, OUT_16_PULLDOWN_RESISTOR, OUT_16_PULLUP_RESISTOR, OUT_17_PULLDOWN_RES, OUT_17_PULLUP_RES, OUT_18_PULLUP_RES, OUT_18_TO_PULLDOWN_RES, OUT_1_PULLDOWN_RES, OUT_1_PULLUP_RES, OUT_1_PULLUP_RES2, OUT_1_PULLUP_RES8, OUT_2_PULLDOWN_RES, OUT_3_PULLDOWN_RES, OUT_4_PULLDOWN_RES, OUT_4_PULLUP_RES, OUT_5_PULLDOWN_RES, OUT_5_PULLUP_RES, OUT_6_PULLDOWN_RES, OUT_6_PULLUP_RES, OUT_7_PULLDOWN_RES, OUT_7_PULLUP_RES, OUT_8_PULLDOWN_RES, OUT_8_PULLUP_RES, OUT_9_PULLDOWN_RES, OUT_9_PULLUP_RES: (no value), rcl:0204/7
- added J35, J36, J37, J38, J39, J40, J41, J42: (no value), SparkFun-Connectors:1X16
- added MOSFET_15, MOSFET_19, MOSFET_20, MOSFET_21, MOSFET_22, MOSFET_23, MOSFET_24: (no value), SparkFun-Connectors:1X03
- added OUT_19_TO_SINGLE, OUT_20_BYPASS, OUT_20_TO_SINGLE, OUT_21_BYPASS, OUT_21_TO_SINGLE, OUT_22_BYPASS, OUT_22_TO_SINGLE, OUT_23_BYPASS, OUT_23_TO_SINGLE, OUT_24_BYPASS, OUT_24_TO_SINGLE, OUT_BYPASS_19, SHFT_TO_SIGNAL_01, SHFT_TO_SIGNAL_02, SHFT_TO_SIGNAL_03, SHFT_TO_SIGNAL_04, SHFT_TO_SIGNAL_05, SHFT_TO_SIGNAL_06, SHFT_TO_SIGNAL_07, SHFT_TO_SIGNAL_08, SHFT_TO_SIGNAL_09, SHFT_TO_SIGNAL_10, SHFT_TO_SIGNAL_11, SHFT_TO_SIGNAL_12, SHFT_TO_SIGNAL_13, SHFT_TO_SIGNAL_14, SHFT_TO_SIGNAL_15, SHFT_TO_SIGNAL_16, TLC_TO_SIGNAL_01, TLC_TO_SIGNAL_02, TLC_TO_SIGNAL_03, TLC_TO_SIGNAL_04, TLC_TO_SIGNAL_05, TLC_TO_SIGNAL_06, TLC_TO_SIGNAL_07, TLC_TO_SIGNAL_08, TLC_TO_SIGNAL_09, TLC_TO_SIGNAL_10, TLC_TO_SIGNAL_11, TLC_TO_SIGNAL_12, TLC_TO_SIGNAL_13, TLC_TO_SIGNAL_14, TLC_TO_SIGNAL_15, TLC_TO_SIGNAL_16: (no value), jumper:SJ
- added RES_I01, RES_I02, RES_I03, RES_I04, RES_I05, RES_I06, RES_I07, RES_I08, RES_I09, RES_I10, RES_I11, RES_I12, RES_I13, RES_I14, RES_I15, RES_I16, RES_I17, RES_I18, RES_I19, RES_I20, RES_I21, RES_I22, RES_I23, RES_I24, RES_O01, RES_O02, RES_O03, RES_O04, RES_O05, RES_O06, RES_O07, RES_O08, RES_O09, RES_O10, RES_O11, RES_O12, RES_O13, RES_O14, RES_O15, RES_O16, RES_O17, RES_O18, RES_O19, RES_O20, RES_O21, RES_O22, RES_O23, RES_O24: (no value), rcl:0204/7
- moved D12_TINY1_GEN_1 908.3 mm to (129.5, -17.8)
- moved D4_TO_SHFT_RCK 908.3 mm to (129.5, -83.8)
- moved D6_TO_SHFT_OE 908.3 mm to (129.5, -99.1)
- moved D9_GEN_4 908.3 mm to (129.5, -43.2)
- moved GEN_1_TO_TLC_GSCLK 908.3 mm to (129.5, -114.3)
- moved GEN_2_TO_SHFT_RCK 908.3 mm to (129.5, -58.4)
- moved GND_TO_SHFT_OE 908.3 mm to (129.5, -73.7)
- moved MOSFET_05 908.3 mm to (229.9, 5.08)
- moved MOSFET_06 908.3 mm to (247.7, 5.08)
- moved MOSFET_13 908.3 mm to (238.8, 5.08)
- moved MOSFET_14 908.3 mm to (256.5, 5.08)
- moved OUT_13_TO_SINGLE 908.3 mm to (129.5, 146.1)
- moved OUT_14_TO_SINGLE 908.3 mm to (170.2, 146.1)
- moved OUT_15_TO_SINGLE 908.3 mm to (129.5, 141.0)
- moved OUT_16_TO_SINGLE 908.3 mm to (170.2, 141.0)
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Connections:
- new net N$100: J41.13, J42.13
- new net N$101: J41.12, J42.12
- new net N$102: J41.11, J42.11
- new net N$103: J41.10, J42.10
- new net N$104: J41.9, J42.9
- new net N$105: J41.8, J42.8
- new net N$106: J41.7, J42.7
- new net N$107: J41.6, J42.6
- new net N$108: J41.5, J42.5
- new net N$109: J41.4, J42.4
- new net N$110: J41.3, J42.3
- new net N$111: J41.2, J42.2
- new net N$112: J41.1, J42.1
- new net N$18: MOSFET_19.1, OUT_19_TO_SINGLE.2, RES_I19.1
- new net N$61: MOSFET_20.1, OUT_20_TO_SINGLE.2, RES_I20.1
- new net N$65: MOSFET_21.1, OUT_21_TO_SINGLE.2, RES_I21.1
- new net N$75: MOSFET_22.1, OUT_22_TO_SINGLE.2, RES_I22.1
- new net N$77: MOSFET_23.1, OUT_23_TO_SINGLE.2, RES_I23.1
- new net N$79: MOSFET_24.1, OUT_24_TO_SINGLE.2, RES_I24.1
- new net N$81: J39.16, J40.16
- new net N$82: J39.15, J40.15
- new net N$83: J39.14, J40.14
- new net N$84: J39.13, J40.13
- new net N$85: J39.12, J40.12
- new net N$86: J39.11, J40.11
- new net N$87: J39.10, J40.10
- new net N$88: J39.9, J40.9
- new net N$89: J39.8, J40.8
- new net N$90: J39.7, J40.7
- new net N$91: J39.6, J40.6
- new net N$92: J39.5, J40.5
- new net N$93: J39.4, J40.4
- new net N$94: J39.3, J40.3
- new net N$95: J39.2, J40.2
- new net N$96: J39.1, J40.1
- new net N$97: J41.16, J42.16
- new net N$98: J41.15, J42.15
- new net N$99: J41.14, J42.14
- new net OUT_FINAL_02: J35.3, J36.3
- new net OUT_FINAL_16: J37.6, J38.6, MOSFET_16.2, OUT_16_BYPASS.1, RES_O16.1
- new net OUT_FINAL_19: J37.10, J38.10, MOSFET_19.2, OUT_BYPASS_19.1, RES_O19.1
- new net OUT_FINAL_20: J37.11, J38.11, MOSFET_20.2, OUT_20_BYPASS.1, RES_O20.1
- new net OUT_FINAL_21: J37.12, J38.12, MOSFET_21.2, OUT_21_BYPASS.1, RES_O21.1
- new net OUT_FINAL_22: J37.14, J38.14, MOSFET_22.2, OUT_22_BYPASS.1, RES_O22.1
- new net OUT_FINAL_23: J37.15, J38.15, MOSFET_23.2, OUT_23_BYPASS.1, RES_O23.1
- new net OUT_FINAL_24: J37.16, J38.16, MOSFET_24.2, OUT_24_BYPASS.1, RES_O24.1
- new net SHFT_OUT_SIGNAL_01: SHFT_TO_SIGNAL_01.2
- new net SHFT_OUT_SIGNAL_02: SHFT_TO_SIGNAL_02.2
- new net SHFT_OUT_SIGNAL_03: SHFT_TO_SIGNAL_03.2
- new net SHFT_OUT_SIGNAL_04: SHFT_TO_SIGNAL_04.2
- new net SHFT_OUT_SIGNAL_05: SHFT_TO_SIGNAL_05.2
- new net SHFT_OUT_SIGNAL_06: SHFT_TO_SIGNAL_06.2
- new net SHFT_OUT_SIGNAL_07: SHFT_TO_SIGNAL_07.2
- new net SHFT_OUT_SIGNAL_08: SHFT_TO_SIGNAL_08.2
- new net SHFT_OUT_SIGNAL_09: SHFT_TO_SIGNAL_09.2
- new net SHFT_OUT_SIGNAL_10: SHFT_TO_SIGNAL_10.2
- new net SHFT_OUT_SIGNAL_11: SHFT_TO_SIGNAL_11.2
- new net SHFT_OUT_SIGNAL_12: SHFT_TO_SIGNAL_12.2
- new net SHFT_OUT_SIGNAL_13: SHFT_TO_SIGNAL_13.2
- new net SHFT_OUT_SIGNAL_14: SHFT_TO_SIGNAL_14.2
- new net SHFT_OUT_SIGNAL_15: SHFT_TO_SIGNAL_15.2
- new net SHFT_OUT_SIGNAL_16: SHFT_TO_SIGNAL_16.2
- new net TLC_OUT_SIGNAL_01: TLC_TO_SIGNAL_01.1
- new net TLC_OUT_SIGNAL_02: TLC_TO_SIGNAL_02.1
- new net TLC_OUT_SIGNAL_03: TLC_TO_SIGNAL_03.1
- new net TLC_OUT_SIGNAL_04: TLC_TO_SIGNAL_04.1
- new net TLC_OUT_SIGNAL_05: TLC_TO_SIGNAL_05.1
- new net TLC_OUT_SIGNAL_06: TLC_TO_SIGNAL_06.1
- new net TLC_OUT_SIGNAL_07: TLC_TO_SIGNAL_07.1
- new net TLC_OUT_SIGNAL_08: TLC_TO_SIGNAL_08.1
- new net TLC_OUT_SIGNAL_09: TLC_TO_SIGNAL_09.1
- new net TLC_OUT_SIGNAL_10: TLC_TO_SIGNAL_10.1
- new net TLC_OUT_SIGNAL_11: TLC_TO_SIGNAL_11.1
- new net TLC_OUT_SIGNAL_12: TLC_TO_SIGNAL_12.1
- new net TLC_OUT_SIGNAL_13: TLC_TO_SIGNAL_13.1
- new net TLC_OUT_SIGNAL_14: TLC_TO_SIGNAL_14.1
- new net TLC_OUT_SIGNAL_15: TLC_TO_SIGNAL_15.1
- new net TLC_OUT_SIGNAL_16: TLC_TO_SIGNAL_16.1
- net +5V: now also RES_I01.2, RES_I02.2, RES_I03.2, RES_I04.2, RES_I05.2, RES_I06.2, RES_I07.2, RES_I08.2, RES_I09.2, RES_I10.2, RES_I11.2, RES_I12.2, RES_I13.2, RES_I14.2, RES_I15.2, RES_I16.2, RES_I17.2, RES_I18.2, RES_I19.2, RES_I20.2, RES_I21.2, RES_I22.2, RES_I23.2, RES_I24.2
- net GND: now also MOSFET_15.3, MOSFET_19.3, MOSFET_20.3, MOSFET_21.3, MOSFET_22.3, MOSFET_23.3, MOSFET_24.3; no longer MOSFET-15.3, OUT_10_PULLDOWN_RES.2, OUT_11_PULLDOWN_RES.2, OUT_12_PULLDOWN_RES.2, OUT_13_PULLDOWN_RES.2, OUT_14_PULLDOWN_RES.2, OUT_15_PULLDOWN_RES.2, OUT_16_PULLDOWN_RESISTOR.2, OUT_17_PULLDOWN_RES.2, OUT_18_TO_PULLDOWN_RES.2, OUT_1_PULLDOWN_RES.2, OUT_2_PULLDOWN_RES.2, OUT_3_PULLDOWN_RES.2, OUT_4_PULLDOWN_RES.2, OUT_5_PULLDOWN_RES.2, OUT_6_PULLDOWN_RES.2, OUT_7_PULLDOWN_RES.2, OUT_8_PULLDOWN_RES.2, OUT_9_PULLDOWN_RES.2
- net N$178: now also RES_I05.1; no longer OUT_5_PULLDOWN_RES.1
- net N$180: now also RES_I13.1; no longer OUT_13_PULLDOWN_RES.1
- net N$182: now also RES_I06.1; no longer OUT_6_PULLDOWN_RES.1
- net N$184: now also RES_I14.1; no longer OUT_14_PULLDOWN_RES.1
- net N$194: now also RES_I07.1; no longer OUT_7_PULLDOWN_RES.1
- net N$196: now also MOSFET_15.1, RES_I15.1; no longer MOSFET-15.1, OUT_15_PULLDOWN_RES.1
- net N$198: now also RES_I08.1; no longer OUT_8_PULLDOWN_RES.1
- net N$200: now also RES_I16.1; no longer OUT_16_PULLDOWN_RESISTOR.1
- net N$50: now also RES_I01.1; no longer OUT_1_PULLDOWN_RES.1
- net N$51: now also RES_I09.1; no longer OUT_9_PULLDOWN_RES.1
- net N$54: now also RES_I02.1; no longer OUT_2_PULLDOWN_RES.1
- net N$56: now also RES_I10.1; no longer OUT_10_PULLDOWN_RES.1
- net N$58: now also RES_I17.1; no longer OUT_17_PULLDOWN_RES.1
- net N$62: now also RES_I18.1; no longer OUT_18_TO_PULLDOWN_RES.1
- net N$66: now also RES_I03.1; no longer OUT_3_PULLDOWN_RES.1
- net N$68: now also RES_I11.1; no longer OUT_11_PULLDOWN_RES.1
- net N$70: now also RES_I04.1; no longer OUT_4_PULLDOWN_RES.1
- net N$72: now also RES_I12.1; no longer OUT_12_PULLDOWN_RES.1
- net OUT_FINAL_01: now also J35.2, J36.2, RES_O01.1; no longer OUT_1_PULLUP_RES.1
- net OUT_FINAL_03: now also J35.4, J36.4, RES_O03.1; no longer OUT_1_PULLUP_RES8.1
- net OUT_FINAL_04: now also J35.6, J36.6, RES_O04.1; no longer OUT_4_PULLUP_RES.1
- net OUT_FINAL_05: now also J35.7, J36.7, RES_O05.1; no longer OUT_5_PULLUP_RES.1
- net OUT_FINAL_06: now also J35.8, J36.8, RES_O06.1; no longer OUT_6_PULLUP_RES.1
- net OUT_FINAL_07: now also J35.10, J36.10, RES_O07.1; no longer OUT_7_PULLUP_RES.1
- net OUT_FINAL_08: now also J35.11, J36.11, RES_O08.1; no longer OUT_8_PULLUP_RES.1
- net OUT_FINAL_09: now also J35.12, J36.12, RES_O09.1; no longer OUT_9_PULLUP_RES.1
- net OUT_FINAL_10: now also J35.14, J36.14, RES_O10.1; no longer OUT_10_PULLUP_RES.1
- net OUT_FINAL_11: now also J35.15, J36.15, RES_O11.1; no longer OUT_11_PULLUP_RES.1
- net OUT_FINAL_12: now also J35.16, J36.16, RES_O12.1; no longer OUT_12_PULLUP_RES.1
- net OUT_FINAL_13: now also J37.2, J38.2, RES_O13.1; no longer OUT_13_PULLUP_RES.1
- net OUT_FINAL_14: now also J37.3, J38.3, RES_O14.1; no longer OUT_14_PULLUP_RES.1
- net OUT_FINAL_15: now also J37.4, J38.4, MOSFET_15.2, RES_O15.1; no longer MOSFET-15.2, OUT_15_PULLUP_RES.1
- net OUT_FINAL_17: now also J37.7, J38.7, RES_O17.1; no longer OUT_17_PULLUP_RES.1
- net OUT_FINAL_18: now also J37.8, J38.8, RES_O18.1; no longer OUT_18_PULLUP_RES.1
- net OUT_PWR: now also J24.1, J24.13, J24.5, J24.9, J25.1, J25.13, J25.5, J25.9, J26.1, J26.13, J26.5, J26.9, J27.1, J27.13, J27.5, J27.9, J35.1, J35.13, J35.5, J35.9, J36.1, J36.13, J36.5, J36.9, J37.1, J37.13, J37.5, J37.9, J38.1, J38.13, J38.5, J38.9, RES_O01.2, RES_O02.2, RES_O03.2, RES_O04.2, RES_O05.2, RES_O06.2, RES_O07.2, RES_O08.2, RES_O09.2, RES_O10.2, RES_O11.2, RES_O12.2, RES_O13.2, RES_O14.2, RES_O15.2, RES_O16.2, RES_O17.2, RES_O18.2, RES_O19.2, RES_O20.2, RES_O21.2, RES_O22.2, RES_O23.2, RES_O24.2; no longer OUT_10_PULLUP_RES.2, OUT_11_PULLUP_RES.2, OUT_12_PULLUP_RES.2, OUT_13_PULLUP_RES.2, OUT_14_PULLUP_RES.2, OUT_15_PULLUP_RES.2, OUT_16_PULLUP_RESISTOR.2, OUT_17_PULLUP_RES.2, OUT_18_PULLUP_RES.2, OUT_1_PULLUP_RES.2, OUT_1_PULLUP_RES2.2, OUT_1_PULLUP_RES8.2, OUT_4_PULLUP_RES.2, OUT_5_PULLUP_RES.2, OUT_6_PULLUP_RES.2, OUT_7_PULLUP_RES.2, OUT_8_PULLUP_RES.2, OUT_9_PULLUP_RES.2
- net OUT_SIGNAL_01: now also SHFT_TO_SIGNAL_01.1, TLC_TO_SIGNAL_01.2
- net OUT_SIGNAL_02: now also SHFT_TO_SIGNAL_02.1, TLC_TO_SIGNAL_02.2
- net OUT_SIGNAL_03: now also SHFT_TO_SIGNAL_03.1, TLC_TO_SIGNAL_03.2
- net OUT_SIGNAL_04: now also SHFT_TO_SIGNAL_04.1, TLC_TO_SIGNAL_04.2
- net OUT_SIGNAL_05: now also SHFT_TO_SIGNAL_05.1, TLC_TO_SIGNAL_05.2
- net OUT_SIGNAL_06: now also SHFT_TO_SIGNAL_06.1, TLC_TO_SIGNAL_06.2
- net OUT_SIGNAL_07: now also SHFT_TO_SIGNAL_07.1, TLC_TO_SIGNAL_07.2
- net OUT_SIGNAL_08: now also SHFT_TO_SIGNAL_08.1, TLC_TO_SIGNAL_08.2
- net OUT_SIGNAL_09: now also SHFT_TO_SIGNAL_09.1, TLC_TO_SIGNAL_09.2
- net OUT_SIGNAL_10: now also SHFT_TO_SIGNAL_10.1, TLC_TO_SIGNAL_10.2
- net OUT_SIGNAL_11: now also SHFT_TO_SIGNAL_11.1, TLC_TO_SIGNAL_11.2
- net OUT_SIGNAL_12: now also SHFT_TO_SIGNAL_12.1, TLC_TO_SIGNAL_12.2
- net OUT_SIGNAL_13: now also SHFT_TO_SIGNAL_13.1, TLC_TO_SIGNAL_13.2
- net OUT_SIGNAL_14: now also SHFT_TO_SIGNAL_14.1, TLC_TO_SIGNAL_14.2
- net OUT_SIGNAL_15: now also SHFT_TO_SIGNAL_15.1, TLC_TO_SIGNAL_15.2
- net OUT_SIGNAL_16: now also SHFT_TO_SIGNAL_16.1, TLC_TO_SIGNAL_16.2; no longer MOSFET_16.2, OUT_16_BYPASS.1, OUT_16_PULLUP_RESISTOR.1
- net OUT_SIGNAL_19: now also OUT_19_TO_SINGLE.1, OUT_BYPASS_19.2
- net OUT_SIGNAL_2: now also RES_O02.1; no longer OUT_1_PULLUP_RES2.1
- net OUT_SIGNAL_20: now also OUT_20_BYPASS.2, OUT_20_TO_SINGLE.1
- net OUT_SIGNAL_21: now also OUT_21_BYPASS.2, OUT_21_TO_SINGLE.1
- net OUT_SIGNAL_22: now also OUT_22_BYPASS.2, OUT_22_TO_SINGLE.1
- net OUT_SIGNAL_23: now also OUT_23_BYPASS.2, OUT_23_TO_SINGLE.1
- net OUT_SIGNAL_24: now also OUT_24_BYPASS.2, OUT_24_TO_SINGLE.1
- net OUT_SIGNAL_25: now also J24.2, J25.2
- net OUT_SIGNAL_26: now also J24.3, J25.3
- net OUT_SIGNAL_27: now also J24.4, J25.4
- net OUT_SIGNAL_28: now also J24.6, J25.6
- net OUT_SIGNAL_29: now also J24.7, J25.7
- net OUT_SIGNAL_30: now also J24.8, J25.8
- net OUT_SIGNAL_31: now also J24.10, J25.10
- net OUT_SIGNAL_32: now also J24.11, J25.11
- net OUT_SIGNAL_33: now also J24.12, J25.12
- net OUT_SIGNAL_34: now also J24.14, J25.14
- net OUT_SIGNAL_35: now also J24.15, J25.15
- net OUT_SIGNAL_36: now also J24.16, J25.16
- net OUT_SIGNAL_37: now also J26.2, J27.2
- net OUT_SIGNAL_38: now also J26.3, J27.3
- net OUT_SIGNAL_39: now also J26.4, J27.4
- net OUT_SIGNAL_40: now also J26.6, J27.6
- net OUT_SIGNAL_41: now also J26.7, J27.7
- net OUT_SIGNAL_42: now also J26.8, J27.8
- net OUT_SIGNAL_43: now also J26.10, J27.10
- net OUT_SIGNAL_44: now also J26.11, J27.11
- net OUT_SIGNAL_45: now also J26.12, J27.12
- net OUT_SIGNAL_46: now also J26.14, J27.14
- net OUT_SIGNAL_47: now also J26.15, J27.15
- net OUT_SIGNAL_48: now also J26.16, J27.16

Commit message: so so close
Parts:
- removed J28, J29, J30, J31, J32, J33, J34: (no value), SparkFun-Connectors:1X30
- removed MOSFET_10, MOSFET_11, MOSFET_12, MOSFET_13, MOSFET_14, MOSFET_15, MOSFET_16, MOSFET_17, MOSFET_18, MOSFET_19, MOSFET_20, MOSFET_21, MOSFET_22, MOSFET_23, MOSFET_24: (no value), SparkFun-Connectors:1X03
- removed OUT_10_BYPASS, OUT_10_TO_SIGNLE, OUT_11_BYPASS, OUT_11_TO_SINGLE, OUT_12_BYPASS, OUT_12_TO_SINGLE, OUT_13_BYPASS, OUT_13_TO_SINGLE, OUT_14_BYPASS, OUT_14_TO_SINGLE, OUT_15_BYPASS, OUT_15_TO_SINGLE, OUT_16_BYPASS, OUT_16_TO_SINGLE, OUT_17_TO_SINGLE, OUT_18_BYPASS, OUT_18_TO_SINGLE, OUT_19_TO_SINGLE, OUT_1_TO_SINGLE1, OUT_20_BYPASS, OUT_20_TO_SINGLE, OUT_21_BYPASS, OUT_21_TO_SINGLE, OUT_22_BYPASS, OUT_22_TO_SINGLE, OUT_23_BYPASS, OUT_23_TO_SINGLE, OUT_24_BYPASS, OUT_24_TO_SINGLE, OUT_BYPASS_17, OUT_BYPASS_19, OUT_PWR_TO_12V_2, OUT_PWR_TO_12V_3, OUT_PWR_TO_12V_4, OUT_PWR_TO_5V_2, OUT_PWR_TO_5V_3, OUT_PWR_TO_5V_4: (no value), jumper:SJ
- removed RES_I10, RES_I11, RES_I12, RES_I13, RES_I14, RES_I15, RES_I16, RES_I17, RES_I18, RES_I19, RES_I20, RES_I21, RES_I22, RES_I23, RES_I24, RES_O10, RES_O11, RES_O12, RES_O13, RES_O14, RES_O15, RES_O16, RES_O17, RES_O18, RES_O19, RES_O20, RES_O21, RES_O22, RES_O23, RES_O24: (no value), rcl:0204/7
- added J43, J44, J45, J46: (no value), SparkFun-Connectors:SCREWTERMINAL-5MM-2
- added OUT_9_TO_SINGLE, OUT_PWR_TO_VIN: (no value), jumper:SJ
- moved SHFT_TO_SIGNAL_01 241.8 mm to (91.4, 78.7)
- moved TLC_TO_SIGNAL_01 236.8 mm to (91.4, 78.7), flipped to the bottom, turned to 180 degrees
- moved GEN_3_TO_TLC_XLAT 224.6 mm to (52.1, 86.4), flipped to the bottom
- moved D6_TO_SHFT_OE 223.5 mm to (12.7, 91.4), flipped to the bottom
- moved GEN_2_TO_TLC_SCLK 220.9 mm to (77.5, 80.0), flipped to the bottom
- moved D3_TO_TLC_GSCLK 220.5 mm to (57.1, 88.9), flipped to the bottom
- moved OUT_5_SINGLE 210.9 mm to (96.5, 48.3), flipped to the bottom, turned to 180 degrees
- moved D5_TO_SHFT_SCL 210.6 mm to (12.7, 81.3), flipped to the bottom
- moved OUT_7_TO_SINGLE 208.5 mm to (96.5, 33.0), flipped to the bottom, turned to 180 degrees
- moved D3_TO_SHFT_SCK 208.5 mm to (12.7, 83.8), flipped to the bottom
- moved GEN_1_TO_TLC_GSCLK 208.0 mm to (74.9, 86.4), flipped to the bottom
- moved D4_TO_SHFT_RCK 206.4 mm to (12.7, 86.4), flipped to the bottom
- moved GEN_3_TO_TLC_BLANK 206.4 mm to (63.5, 86.4), flipped to the bottom
- moved D2_TO_SHFT_SER_IN 204.3 mm to (12.7, 88.9), flipped to the bottom
- moved GEN_0_TO_TLC_SIN 202.4 mm to (68.6, 88.9), flipped to the bottom
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Connections:
- removed net N$10: J31.25, J31.26, J31.27
- removed net N$100: J41.13, J42.13
- removed net N$101: J41.12, J42.12
- removed net N$102: J41.11, J42.11
- removed net N$103: J41.10, J42.10
- removed net N$104: J41.9, J42.9
- removed net N$105: J41.8, J42.8
- removed net N$106: J41.7, J42.7
- removed net N$107: J41.6, J42.6
- removed net N$108: J41.5, J42.5
- removed net N$109: J41.4, J42.4
- removed net N$110: J41.3, J42.3
- removed net N$111: J41.2, J42.2
- removed net N$112: J41.1, J42.1
- removed net N$13: J32.25, J32.26, J32.27
- removed net N$16: J32.22, J32.23, J32.24
- removed net N$17: J31.22, J31.23, J31.24
- removed net N$18: MOSFET_19.1, OUT_19_TO_SINGLE.2, RES_I19.1
- removed net N$180: MOSFET_13.1, OUT_13_TO_SINGLE.2, RES_I13.1
- removed net N$184: MOSFET_14.1, OUT_14_TO_SINGLE.2, RES_I14.1
- removed net N$19: J30.22, J30.23, J30.24
- removed net N$196: MOSFET_15.1, OUT_15_TO_SINGLE.2, RES_I15.1
- removed net N$2: J29.28, J29.29, J29.30
- removed net N$20: J29.22, J29.23, J29.24
- removed net N$200: MOSFET_16.1, OUT_16_TO_SINGLE.2, RES_I16.1
- removed net N$22: J29.19, J29.20, J29.21
- removed net N$23: J30.19, J30.20, J30.21
- removed net N$24: J31.19, J31.20, J31.21
- removed net N$25: J32.19, J32.20, J32.21
- removed net N$26: J32.16, J32.17, J32.18
- removed net N$27: J31.16, J31.17, J31.18
- removed net N$28: J30.16, J30.17, J30.18
- removed net N$29: J29.16, J29.17, J29.18
- removed net N$3: J30.28, J30.29, J30.30
- removed net N$30: J29.13, J29.14, J29.15
- removed net N$31: J30.13, J30.14, J30.15
- removed net N$32: J31.13, J31.14, J31.15
- removed net N$33: J32.13, J32.14, J32.15
- removed net N$34: J32.10, J32.11, J32.12
- removed net N$35: J31.10, J31.11, J31.12
- removed net N$36: J30.10, J30.11, J30.12
- removed net N$37: J29.10, J29.11, J29.12
- removed net N$38: J32.7, J32.8, J32.9
- removed net N$39: J32.4, J32.5, J32.6
- removed net N$4: J31.28, J31.29, J31.30
- removed net N$40: J32.1, J32.2, J32.3
- removed net N$41: J31.7, J31.8, J31.9
- removed net N$42: J31.4, J31.5, J31.6
- removed net N$43: J31.1, J31.2, J31.3
- removed net N$44: J30.7, J30.8, J30.9
- removed net N$45: J30.4, J30.5, J30.6
- removed net N$46: J30.1, J30.2, J30.3
- removed net N$47: J29.7, J29.8, J29.9
- removed net N$48: J29.4, J29.5, J29.6
- removed net N$49: J29.1, J29.2, J29.3
- removed net N$56: MOSFET_10.1, OUT_10_TO_SIGNLE.2, RES_I10.1
- removed net N$58: MOSFET_17.1, OUT_17_TO_SINGLE.2, RES_I17.1
- removed net N$61: MOSFET_20.1, OUT_20_TO_SINGLE.2, RES_I20.1
- removed net N$62: MOSFET_18.1, OUT_18_TO_SINGLE.2, RES_I18.1
- removed net N$65: MOSFET_21.1, OUT_21_TO_SINGLE.2, RES_I21.1
- removed net N$68: MOSFET_11.1, OUT_11_TO_SINGLE.2, RES_I11.1
- removed net N$7: J32.28, J32.29, J32.30
- removed net N$72: MOSFET_12.1, OUT_12_TO_SINGLE.2, RES_I12.1
- removed net N$75: MOSFET_22.1, OUT_22_TO_SINGLE.2, RES_I22.1
- removed net N$77: MOSFET_23.1, OUT_23_TO_SINGLE.2, RES_I23.1
- removed net N$79: MOSFET_24.1, OUT_24_TO_SINGLE.2, RES_I24.1
- removed net N$8: J29.25, J29.26, J29.27
- removed net N$81: J39.16, J40.16
- removed net N$82: J39.15, J40.15
- removed net N$83: J39.14, J40.14
- removed net N$84: J39.13, J40.13
- removed net N$85: J39.12, J40.12
- removed net N$86: J39.11, J40.11
- removed net N$87: J39.10, J40.10
- removed net N$88: J39.9, J40.9
- removed net N$89: J39.8, J40.8
- removed net N$9: J30.25, J30.26, J30.27
- removed net N$90: J39.7, J40.7
- removed net N$91: J39.6, J40.6
- removed net N$92: J39.5, J40.5
- removed net N$93: J39.4, J40.4
- removed net N$94: J39.3, J40.3
- removed net N$95: J39.2, J40.2
- removed net N$96: J39.1, J40.1
- removed net N$97: J41.16, J42.16
- removed net N$98: J41.15, J42.15
- removed net N$99: J41.14, J42.14
- removed net OUT_FINAL_10: J35.14, J36.14, MOSFET_10.2, OUT_10_BYPASS.1, RES_O10.1
- removed net OUT_FINAL_11: J35.15, J36.15, MOSFET_11.2, OUT_11_BYPASS.1, RES_O11.1
- removed net OUT_FINAL_12: J35.16, J36.16, MOSFET_12.2, OUT_12_BYPASS.1, RES_O12.1
- removed net OUT_FINAL_13: J37.2, J38.2, MOSFET_13.2, OUT_13_BYPASS.1, RES_O13.1
- removed net OUT_FINAL_14: J37.3, J38.3, MOSFET_14.2, OUT_14_BYPASS.1, RES_O14.1
- removed net OUT_FINAL_15: J37.4, J38.4, MOSFET_15.2, OUT_15_BYPASS.1, RES_O15.1
- removed net OUT_FINAL_16: J37.6, J38.6, MOSFET_16.2, OUT_16_BYPASS.1, RES_O16.1
- removed net OUT_FINAL_17: J37.7, J38.7, MOSFET_17.2, OUT_BYPASS_17.1, RES_O17.1
- removed net OUT_FINAL_18: J37.8, J38.8, MOSFET_18.2, OUT_18_BYPASS.1, RES_O18.1
- removed net OUT_FINAL_19: J37.10, J38.10, MOSFET_19.2, OUT_BYPASS_19.1, RES_O19.1
- removed net OUT_FINAL_20: J37.11, J38.11, MOSFET_20.2, OUT_20_BYPASS.1, RES_O20.1
- removed net OUT_FINAL_21: J37.12, J38.12, MOSFET_21.2, OUT_21_BYPASS.1, RES_O21.1
- removed net OUT_FINAL_22: J37.14, J38.14, MOSFET_22.2, OUT_22_BYPASS.1, RES_O22.1
- removed net OUT_FINAL_23: J37.15, J38.15, MOSFET_23.2, OUT_23_BYPASS.1, RES_O23.1
- removed net OUT_FINAL_24: J37.16, J38.16, MOSFET_24.2, OUT_24_BYPASS.1, RES_O24.1
- removed net OUT_SIGNAL_2: MOSFET_02.2, OUT_2_BYPASS.1, RES_O02.1
- net +12V: no longer OUT_PWR_TO_12V_2.2, OUT_PWR_TO_12V_3.2, OUT_PWR_TO_12V_4.2
- net +5V: no longer J34.1, J34.10, J34.11, J34.12, J34.13, J34.14, J34.15, J34.16, J34.17, J34.18, J34.19, J34.2, J34.20, J34.21, J34.22, J34.23, J34.24, J34.25, J34.26, J34.27, J34.28, J34.29, J34.3, J34.30, J34.4, J34.5, J34.6, J34.7, J34.8, J34.9, OUT_PWR_TO_5V_2.2, OUT_PWR_TO_5V_3.2, OUT_PWR_TO_5V_4.2, RES_I10.2, RES_I11.2, RES_I12.2, RES_I13.2, RES_I14.2, RES_I15.2, RES_I16.2, RES_I17.2, RES_I18.2, RES_I19.2, RES_I20.2, RES_I21.2, RES_I22.2, RES_I23.2, RES_I24.2
- net GND: now also J43.1, J44.1, J45.1, J46.1; no longer J33.1, J33.10, J33.11, J33.12, J33.13, J33.14, J33.15, J33.16, J33.17, J33.18, J33.19, J33.2, J33.20, J33.21, J33.22, J33.23, J33.24, J33.25, J33.26, J33.27, J33.28, J33.29, J33.3, J33.30, J33.4, J33.5, J33.6, J33.7, J33.8, J33.9, MOSFET_10.3, MOSFET_11.3, MOSFET_12.3, MOSFET_13.3, MOSFET_14.3, MOSFET_15.3, MOSFET_16.3, MOSFET_17.3, MOSFET_18.3, MOSFET_19.3, MOSFET_20.3, MOSFET_21.3, MOSFET_22.3, MOSFET_23.3, MOSFET_24.3
- net N$51: now also OUT_9_TO_SINGLE.2; no longer OUT_1_TO_SINGLE1.2
- net OUT_FINAL_02: now also MOSFET_02.2, OUT_2_BYPASS.1, RES_O02.1
- net OUT_PWR: now also J43.2, J44.2, J45.2, J46.2, OUT_PWR_TO_VIN.2; no longer J28.1, J28.10, J28.11, J28.12, J28.13, J28.14, J28.15, J28.16, J28.17, J28.18, J28.19, J28.2, J28.20, J28.21, J28.22, J28.23, J28.24, J28.25, J28.26, J28.27, J28.28, J28.29, J28.3, J28.30, J28.4, J28.5, J28.6, J28.7, J28.8, J28.9, OUT_PWR_TO_12V_2.1, OUT_PWR_TO_12V_3.1, OUT_PWR_TO_12V_4.1, OUT_PWR_TO_5V_2.1, OUT_PWR_TO_5V_3.1, OUT_PWR_TO_5V_4.1, RES_O10.2, RES_O11.2, RES_O12.2, RES_O13.2, RES_O14.2, RES_O15.2, RES_O16.2, RES_O17.2, RES_O18.2, RES_O19.2, RES_O20.2, RES_O21.2, RES_O22.2, RES_O23.2, RES_O24.2
- net OUT_SIGNAL_09: now also OUT_9_TO_SINGLE.1; no longer OUT_1_TO_SINGLE1.1
- net OUT_SIGNAL_10: now also J35.14, J36.14; no longer OUT_10_BYPASS.2, OUT_10_TO_SIGNLE.1
- net OUT_SIGNAL_11: now also J35.15, J36.15; no longer OUT_11_BYPASS.2, OUT_11_TO_SINGLE.1
- net OUT_SIGNAL_12: now also J35.16, J36.16; no longer OUT_12_BYPASS.2, OUT_12_TO_SINGLE.1
- net OUT_SIGNAL_13: now also J37.2, J38.2; no longer OUT_13_BYPASS.2, OUT_13_TO_SINGLE.1
- net OUT_SIGNAL_14: now also J37.3, J38.3; no longer OUT_14_BYPASS.2, OUT_14_TO_SINGLE.1
- net OUT_SIGNAL_15: now also J37.4, J38.4; no longer OUT_15_BYPASS.2, OUT_15_TO_SINGLE.1
- net OUT_SIGNAL_16: now also J37.6, J38.6; no longer OUT_16_BYPASS.2, OUT_16_TO_SINGLE.1
- net OUT_SIGNAL_17: now also J37.7, J38.7, SHFT_REG_4.15; no longer OUT_17_TO_SINGLE.1, OUT_BYPASS_17.2, SHFT_REG_3.15
- net OUT_SIGNAL_18: now also J37.8, J38.8, SHFT_REG_4.1; no longer OUT_18_BYPASS.2, OUT_18_TO_SINGLE.1, SHFT_REG_3.1
- net OUT_SIGNAL_19: now also J37.10, J38.10, SHFT_REG_4.2; no longer OUT_19_TO_SINGLE.1, OUT_BYPASS_19.2, SHFT_REG_3.2
- net OUT_SIGNAL_20: now also J37.11, J38.11, SHFT_REG_4.3; no longer OUT_20_BYPASS.2, OUT_20_TO_SINGLE.1, SHFT_REG_3.3
- net OUT_SIGNAL_21: now also J37.12, J38.12, SHFT_REG_4.4; no longer OUT_21_BYPASS.2, OUT_21_TO_SINGLE.1, SHFT_REG_3.4
- net OUT_SIGNAL_22: now also J37.14, J38.14, SHFT_REG_4.5; no longer OUT_22_BYPASS.2, OUT_22_TO_SINGLE.1, SHFT_REG_3.5
- net OUT_SIGNAL_23: now also J37.15, J38.15, SHFT_REG_4.6; no longer OUT_23_BYPASS.2, OUT_23_TO_SINGLE.1, SHFT_REG_3.6
- net OUT_SIGNAL_24: now also J37.16, J38.16, SHFT_REG_4.7; no longer OUT_24_BYPASS.2, OUT_24_TO_SINGLE.1, SHFT_REG_3.7
- net OUT_SIGNAL_25: now also SHFT_REG_3.15; no longer SHFT_REG_4.15
- net OUT_SIGNAL_26: now also SHFT_REG_3.1; no longer SHFT_REG_4.1
- net OUT_SIGNAL_27: now also SHFT_REG_3.2; no longer SHFT_REG_4.2
- net OUT_SIGNAL_28: now also SHFT_REG_3.3; no longer SHFT_REG_4.3
- net OUT_SIGNAL_29: now also SHFT_REG_3.4; no longer SHFT_REG_4.4
- net OUT_SIGNAL_30: now also SHFT_REG_3.5; no longer SHFT_REG_4.5
- net OUT_SIGNAL_31: now also SHFT_REG_3.6; no longer SHFT_REG_4.6
- net OUT_SIGNAL_32: now also SHFT_REG_3.7; no longer SHFT_REG_4.7
- net SHFT_OUT_SIGNAL_01: now also J41.1, J42.1
- net SHFT_OUT_SIGNAL_02: now also J41.2, J42.2
- net SHFT_OUT_SIGNAL_03: now also J41.3, J42.3
- net SHFT_OUT_SIGNAL_04: now also J41.4, J42.4
- net SHFT_OUT_SIGNAL_05: now also J41.5, J42.5
- net SHFT_OUT_SIGNAL_06: now also J41.6, J42.6
- net SHFT_OUT_SIGNAL_07: now also J41.7, J42.7
- net SHFT_OUT_SIGNAL_08: now also J41.8, J42.8
- net SHFT_OUT_SIGNAL_09: now also J41.9, J42.9
- net SHFT_OUT_SIGNAL_10: now also J41.10, J42.10
- net SHFT_OUT_SIGNAL_11: now also J41.11, J42.11
- net SHFT_OUT_SIGNAL_12: now also J41.12, J42.12
- net SHFT_OUT_SIGNAL_13: now also J41.13, J42.13
- net SHFT_OUT_SIGNAL_14: now also J41.14, J42.14
- net SHFT_OUT_SIGNAL_15: now also J41.15, J42.15
- net SHFT_OUT_SIGNAL_16: now also J41.16, J42.16
- net SHFT_REG_2_OUT: now also SHFT_REG_4.14; no longer SHFT_REG_3.14
- net SHFT_REG_3_SOUT: now also SHFT_REG_3.14, SHFT_REG_4.9; no longer SHFT_REG_3.9, SHFT_REG_4.14
- net SHFT_REG_4_SOUT: now also SHFT_REG_3.9; no longer SHFT_REG_4.9
- net TLC_OUT_SIGNAL_01: now also J39.1, J40.1
- net TLC_OUT_SIGNAL_02: now also J39.2, J40.2
- net TLC_OUT_SIGNAL_03: now also J39.3, J40.3
- net TLC_OUT_SIGNAL_04: now also J39.4, J40.4
- net TLC_OUT_SIGNAL_05: now also J39.5, J40.5
- net TLC_OUT_SIGNAL_06: now also J39.6, J40.6
- net TLC_OUT_SIGNAL_07: now also J39.7, J40.7
- net TLC_OUT_SIGNAL_08: now also J39.8, J40.8
- net TLC_OUT_SIGNAL_09: now also J39.9, J40.9
- net TLC_OUT_SIGNAL_10: now also J39.10, J40.10
- net TLC_OUT_SIGNAL_11: now also J39.11, J40.11
- net TLC_OUT_SIGNAL_12: now also J39.12, J40.12
- net TLC_OUT_SIGNAL_13: now also J39.13, J40.13
- net TLC_OUT_SIGNAL_14: now also J39.14, J40.14
- net TLC_OUT_SIGNAL_15: now also J39.15, J40.15
- net TLC_OUT_SIGNAL_16: now also J39.16, J40.16
- net VIN: now also OUT_PWR_TO_VIN.1
Other:
- board text added: "D2"
- board text added: "D3"
- board text added: "D4"
- board text added: "D5"
- board text added: "D6"
- board text added: "GND"
- board text added: "SHFT_OUT_SIGNAL_01"
- board text added: "SHFT_OUT_SIGNAL_16"
- board text added: "TLC CHAIN"
- board text added: "TLC_OUT_SIGNAL_01"
- board text added: "TLC_OUT_SIGNAL_16"

Commit message: multishift ready for auto
Parts:
- removed J45, J46: (no value), SparkFun-Connectors:SCREWTERMINAL-5MM-2
- moved J44 223.3 mm to (31.8, 26.7)
- moved J20 40.6 mm to (19.1, 2.54)
- moved J21 40.6 mm to (19.1, 5.08)
- moved J22 40.6 mm to (59.7, 5.08)
- moved J23 40.6 mm to (59.7, 2.54)
- moved J35 5.08 mm to (13.0, 95.1)
- moved J36 5.08 mm to (13.0, 97.9)
- moved J37 3.81 mm to (53.7, 97.9)
- moved J38 3.81 mm to (53.7, 95.1)
- moved J39 1.27 mm to (25.4, 10.2)
- moved J40 1.27 mm to (25.4, 12.7)
Connections:
- net GND: no longer J45.1, J46.1
- net OUT_PWR: no longer J45.2, J46.2
- net OUT_SIGNAL_01: no longer SHFT_REG_1.15, TLC_1.28
- net OUT_SIGNAL_02: no longer SHFT_REG_1.1, TLC_1.1
- net OUT_SIGNAL_03: no longer SHFT_REG_1.2, TLC_1.2
- net OUT_SIGNAL_04: no longer SHFT_REG_1.3, TLC_1.3
- net OUT_SIGNAL_05: no longer SHFT_REG_1.4, TLC_1.4
- net OUT_SIGNAL_06: no longer SHFT_REG_1.5, TLC_1.5
- net OUT_SIGNAL_07: no longer SHFT_REG_1.6, TLC_1.6
- net OUT_SIGNAL_08: no longer SHFT_REG_1.7, TLC_1.7
- net OUT_SIGNAL_09: no longer SHFT_REG_2.15, TLC_1.8
- net OUT_SIGNAL_10: no longer SHFT_REG_2.1, TLC_1.9
- net OUT_SIGNAL_11: no longer SHFT_REG_2.2, TLC_1.10
- net OUT_SIGNAL_12: no longer SHFT_REG_2.3, TLC_1.11
- net OUT_SIGNAL_13: no longer SHFT_REG_2.4, TLC_1.12
- net OUT_SIGNAL_14: no longer SHFT_REG_2.5, TLC_1.13
- net OUT_SIGNAL_15: no longer SHFT_REG_2.6, TLC_1.14
- net OUT_SIGNAL_16: no longer SHFT_REG_2.7, TLC_1.15
- net SHFT_OUT_SIGNAL_01: now also SHFT_REG_1.15
- net SHFT_OUT_SIGNAL_02: now also SHFT_REG_1.1
- net SHFT_OUT_SIGNAL_03: now also SHFT_REG_1.2
- net SHFT_OUT_SIGNAL_04: now also SHFT_REG_1.3
- net SHFT_OUT_SIGNAL_05: now also SHFT_REG_1.4
- net SHFT_OUT_SIGNAL_06: now also SHFT_REG_1.5
- net SHFT_OUT_SIGNAL_07: now also SHFT_REG_1.6
- net SHFT_OUT_SIGNAL_08: now also SHFT_REG_1.7
- net SHFT_OUT_SIGNAL_09: now also SHFT_REG_2.15
- net SHFT_OUT_SIGNAL_10: now also SHFT_REG_2.1
- net SHFT_OUT_SIGNAL_11: now also SHFT_REG_2.2
- net SHFT_OUT_SIGNAL_12: now also SHFT_REG_2.3
- net SHFT_OUT_SIGNAL_13: now also SHFT_REG_2.4
- net SHFT_OUT_SIGNAL_14: now also SHFT_REG_2.5
- net SHFT_OUT_SIGNAL_15: now also SHFT_REG_2.6
- net SHFT_OUT_SIGNAL_16: now also SHFT_REG_2.7
- net TLC_OUT_SIGNAL_01: now also TLC_1.28
- net TLC_OUT_SIGNAL_02: now also TLC_1.1
- net TLC_OUT_SIGNAL_03: now also TLC_1.2
- net TLC_OUT_SIGNAL_04: now also TLC_1.3
- net TLC_OUT_SIGNAL_05: now also TLC_1.4
- net TLC_OUT_SIGNAL_06: now also TLC_1.5
- net TLC_OUT_SIGNAL_07: now also TLC_1.6
- net TLC_OUT_SIGNAL_08: now also TLC_1.7
- net TLC_OUT_SIGNAL_09: now also TLC_1.8
- net TLC_OUT_SIGNAL_10: now also TLC_1.9
- net TLC_OUT_SIGNAL_11: now also TLC_1.10
- net TLC_OUT_SIGNAL_12: now also TLC_1.11
- net TLC_OUT_SIGNAL_13: now also TLC_1.12
- net TLC_OUT_SIGNAL_14: now also TLC_1.13
- net TLC_OUT_SIGNAL_15: now also TLC_1.14
- net TLC_OUT_SIGNAL_16: now also TLC_1.15
Routing:
- net OUT_SIGNAL_24: track 0.00 -> 5.33 mm
- net OUT_SIGNAL_23: track 0.00 -> 5.33 mm
- net OUT_SIGNAL_22: track 0.00 -> 5.33 mm
- net OUT_SIGNAL_21: track 0.00 -> 5.33 mm
- net OUT_SIGNAL_20: track 0.00 -> 5.33 mm
- net OUT_SIGNAL_19: track 0.00 -> 5.33 mm
- net OUT_SIGNAL_18: track 0.00 -> 5.33 mm
- net OUT_SIGNAL_17: track 0.00 -> 5.33 mm
- net OUT_SIGNAL_16: track 0.00 -> 5.33 mm
- net OUT_SIGNAL_15: track 0.00 -> 5.33 mm
- net OUT_SIGNAL_14: track 0.00 -> 5.33 mm
- net OUT_SIGNAL_13: track 0.00 -> 5.33 mm
- net OUT_SIGNAL_12: track 0.00 -> 5.33 mm
- net OUT_SIGNAL_11: track 0.00 -> 5.33 mm
- net OUT_SIGNAL_10: track 0.00 -> 2.79 mm
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Other:
- board text added: "FINAL_01"
- board text added: "FINAL_02"
- board text added: "FINAL_03"
- board text added: "FINAL_22"
- board text added: "FINAL_23"
- board text added: "FINAL_24"
- board text added: "OUT_PWR"
- board text added: "OUT_PWR...."
- board text added: "OUT_SIGNAL_02"
- board text added: "OUT_SIGNAL_10"
- board text added: "OUT_SIGNAL_19"
- board text added: "OUT_SIGNAL_24"
- board text added: "SIDE: SHFT"
- board text added: "SIGNAL_25"
- board text added: "SIGNAL_48"
- board text added: "TLC SIDE"
